Commit message: save

File: nextage_description/urdf/NextageOpen.urdf (robot description, URDF)
Before this commit: robot NextageOpen, 16 links, 15 joints
Links:
- added link BDU, mass 1000; collision mesh filename=package://nextage_description/urdf/meshes/BDU.stl scale=1 1 1; visual mesh filename=package://nextage_description/urdf/meshes/BDU.stl scale=1 1 1
- added link WORKTABLE, mass 1000; collision mesh filename=package://nextage_description/urdf/meshes/WORKTABLE.stl scale=0.1 0.0 0.1; visual mesh filename=package://nextage_description/urdf/meshes/WORKTABLE.stl scale=0.1 0.1 0.1
Joints:
- added joint BDU_JOINT: type fixed, parent WAIST, child BDU, origin xyz=0 0 0 rpy=0 -0 0 
- added joint WORKTABLE_JOINT: type fixed, parent WAIST, child WORKTABLE, origin xyz=0 0 0 rpy=0 -0 0 

Commit message: add an operator model

File: nextage_description/urdf/NextageOpen.urdf (robot description, URDF)
Before this commit: robot NextageOpen, 18 links, 17 joints
Links:
- removed link BDU
Joints:
- removed joint BDU_JOINT
