Commit message: fix some issues and save a world for gazebo

File: nextage_description/urdf/nxo_gz.xacro (robot description, xacro)
@@ -2,5 +2,5 @@
 <robot name="NextageOpen"
        xmlns:xacro="http://www.ros.org/wiki/xacro">
-  <xacro:include filename="$(find nextage_description)/urdf/NextageOpen.urdf" />
+  <xacro:include filename="$(find nextage_description)/urdf/nxo_world.xacro" />
   <xacro:include filename="$(find nextage_description)/urdf/nxo_gz_camera.xacro" />
   <xacro:property name="M_PI" value="3.1415926535897931" />

File: nextage_description/urdf/nxo_world.xacro (robot description, xacro)
@@ -14,5 +14,5 @@
     <link name="BDU">
         <visual>
-            <origin xyz="0.5 0 -0.08" rpy="0 -0 0"/>
+            <origin xyz="0.75 0 -0.08" rpy="0 -0 0"/>
             <geometry>
                 <mesh filename="package://nextage_description/urdf/meshes/BDU.stl" scale="1 1 1" />
@@ -23,5 +23,5 @@
         </visual>
         <collision>
-            <origin xyz="0.5 0 -0.08" rpy="0 -0 0"/>
+            <origin xyz="0.75 0 -0.08" rpy="0 -0 0"/>
             <geometry>
                 <mesh filename="package://nextage_description/urdf/meshes/BDU.stl" scale="1 1 1" />
@@ -41,4 +41,5 @@
     </joint>
     <!-- operator link with STL mesh -->
+    <xacro:gazebo_nx_link name="OPERATOR" color="Gray" />
     <link name="OPERATOR">
         <visual>
@@ -67,5 +68,5 @@
         <parent link="world"/>
         <child link="OPERATOR"/>
-        <origin xyz="0.5 -0.5 -0.9" rpy="0 0 -1.5708"/>
+        <origin xyz="0.75 -0.5 -1.0" rpy="0 0 -1.5708"/>
     </joint>
 </robot>
