Commit message: save

File: nextage_description/urdf/nxo_world.xacro (robot description, xacro)
@@ -68,5 +68,5 @@
         <parent link="world"/>
         <child link="OPERATOR"/>
-        <origin xyz="0.75 -0.5 -1.0" rpy="0 0 -1.5708"/>
+        <origin xyz="1.5 -0.3 -0.95" rpy="0 0 -0.785398"/>
     </joint>
 </robot>
